File: pcb/Placa_Carrier_ESP32-S3-DEVKIT/Placa_Carrier_ESP32-S3-DEVKIT.kicad_sch (KiCad schematic)
At the start: 0 parts

Commit message: Actualiza sch y PCB
Parts:
- added C1: 100uF/25V, Capacitor_SMD:CP_Elec_6.3x7.7, symbol Device:C_Polarized
- added C2: 22uF/10V, Capacitor_Tantalum_SMD:CP_EIA-3528-21_Kemet-B_Pad1.50x2.35mm_HandSolder, symbol Device:C_Polarized
- added C3, C4, C5: 100nF, Capacitor_SMD:C_0805_2012Metric_Pad1.18x1.45mm_HandSolder, symbol Device:C
- added C6: 10uF/25V, Capacitor_SMD:C_1206_3216Metric_Pad1.33x1.80mm_HandSolder, symbol Device:C
- added D1, D2, D5, D6: SS34, Diode_SMD:D_SMA, symbol Diode:SS34
- added D3, D4, D7: LED, LED_SMD:LED_1206_3216Metric_Pad1.42x1.75mm_HandSolder, symbol Device:LED
- added D8: 1N4148W, Diode_SMD:D_SOD-123, symbol Diode:1N4148W
- added J1: 12V IN, TerminalBlock_Phoenix:TerminalBlock_Phoenix_MKDS-1,5-2-5.08_1x02_P5.08mm_Horizontal, symbol Connector:Screw_Terminal_01x02
- added J2: AN_IN, TerminalBlock_Phoenix:TerminalBlock_Phoenix_MKDS-1,5-3-5.08_1x03_P5.08mm_Horizontal, symbol Connector:Screw_Terminal_01x03
- added J3: RELE, TerminalBlock_Phoenix:TerminalBlock_Phoenix_MKDS-1,5-3-5.08_1x03_P5.08mm_Horizontal, symbol Connector:Screw_Terminal_01x03
- added J4: CAN, TerminalBlock_Phoenix:TerminalBlock_Phoenix_MKDS-1,5-3-5.08_1x03_P5.08mm_Horizontal, symbol Connector:Screw_Terminal_01x03
- added J5: DevKit_J1, Connector_PinSocket_2.54mm:PinSocket_1x22_P2.54mm_Vertical, symbol Connector_Generic:Conn_01x22
- added J6: DevKit_J3, Connector_PinSocket_2.54mm:PinSocket_1x22_P2.54mm_Vertical, symbol Connector_Generic:Conn_01x22
- added J7: EXP_J1, Connector_PinSocket_2.54mm:PinSocket_1x22_P2.54mm_Vertical, symbol Connector_Generic:Conn_01x22
- added J8: EXP_J3, Connector_PinSocket_2.54mm:PinSocket_1x22_P2.54mm_Vertical, symbol Connector_Generic:Conn_01x22
- added JP1: TERM_CAN, Connector_PinHeader_2.54mm:PinHeader_1x02_P2.54mm_Vertical, symbol Jumper:Jumper_2_Open
- added K1: SRD-05VDC, Relay_THT:Relay_SPDT_SANYOU_SRD_Series_Form_C, symbol Relay:SANYOU_SRD_Form_C
- added Q1: BC817, Package_TO_SOT_SMD:SOT-23, symbol Transistor_BJT:BC817
- added R1, R11: 120, Resistor_SMD:R_1206_3216Metric_Pad1.30x1.75mm_HandSolder, symbol Device:R
- added R10, R8: 1k, Resistor_SMD:R_1206_3216Metric_Pad1.30x1.75mm_HandSolder, symbol Device:R
- added R12: 390, Resistor_SMD:R_1206_3216Metric_Pad1.30x1.75mm_HandSolder, symbol Device:R
- added R2, R3: 330, Resistor_SMD:R_1206_3216Metric_Pad1.30x1.75mm_HandSolder, symbol Device:R
- added R4, R5, R7, R9: 10k, Resistor_SMD:R_1206_3216Metric_Pad1.30x1.75mm_HandSolder, symbol Device:R
- added R6: 22k, Resistor_SMD:R_1206_3216Metric_Pad1.30x1.75mm_HandSolder, symbol Device:R
- added SW1, SW2: SW_Push, Button_Switch_THT:SW_PUSH_6mm, symbol Switch:SW_Push
- added U1: AMS1117-ADJ, Package_TO_SOT_SMD:SOT-223-3_TabPin2, symbol Regulator_Linear:AMS1117
- added U3: MCP2562-E-SN, Package_SO:SOIC-8_3.9x4.9mm_P1.27mm, symbol Interface_CAN_LIN:MCP2562-E-SN
Connections:
- new net: R11.2, R12.1, U1.1 (ADJ)
- new net: D7.1 (K), D8.2 (A), K1.2, Q1.3 (C)
- new net: D3.2 (A), R2.2
- new net: Q1.1 (B), R8.2, R9.1
- new net: D7.2 (A), R10.2
- new net: JP1.2 (B), R1.2
- new net: D4.2 (A), R3.2
- new net: J2.2 (Pin_2), R6.1
- new net +12V_IN: D1.2 (A), J1.1 (Pin_1)
- new net +3V3: C4.1, D5.1 (K), J2.1 (Pin_1), J5.1 (Pin_1), J5.2 (Pin_2), J7.1 (Pin_1), J7.2 (Pin_2), R4.1, R5.1, U3.5 (Vio)
- new net +5V: C3.1, D2.1 (K), D8.1 (K), J5.21 (Pin_21), J7.21 (Pin_21), K1.5, R10.1, U3.3 (VDD)
- new net +5V_REG: C2.1, D2.2 (A), R11.1, U1.2 (VO)
- new net AN1: C5.1, D5.2 (A), D6.1 (K), J6.4 (Pin_4), J8.4 (Pin_4), R6.2, R7.1
- new net CANH: J4.1 (Pin_1), R1.1, U3.7 (CANH)
- new net CANL: J4.2 (Pin_2), JP1.1 (A), U3.6 (CANL)
- new net CAN_RX: J5.11 (Pin_11), J7.11 (Pin_11), U3.4 (RXD)
- new net CAN_TX: J5.10 (Pin_10), J7.10 (Pin_10), U3.1 (TXD)
- new net GND: C1.2, C2.2, C3.2, C4.2, C5.2, C6.2, D3.1 (K), D4.1 (K), D6.2 (A), J1.2 (Pin_2), J2.3 (Pin_3), J4.3 (Pin_3), J5.22 (Pin_22), J6.1 (Pin_1), J6.21 (Pin_21), J6.22 (Pin_22), J7.22 (Pin_22), J8.1 (Pin_1), J8.21 (Pin_21), J8.22 (Pin_22), Q1.2 (E), R12.2, R7.2, R9.2, SW1.1, SW2.1, U3.2 (VSS), U3.8 (STBY)
- new net GPIO0: J6.14 (Pin_14), J8.14 (Pin_14)
- new net GPIO11: J5.17 (Pin_17), J7.17 (Pin_17)
- new net GPIO12: J5.18 (Pin_18), J7.18 (Pin_18)
- new net GPIO13: J5.19 (Pin_19), J7.19 (Pin_19)
- new net GPIO14: J5.20 (Pin_20), J7.20 (Pin_20)
- new net GPIO16: J5.9 (Pin_9), J7.9 (Pin_9)
- new net GPIO19: J6.20 (Pin_20), J8.20 (Pin_20)
- new net GPIO2: J6.5 (Pin_5), J8.5 (Pin_5)
- new net GPIO20: J6.19 (Pin_19), J8.19 (Pin_19)
- new net GPIO21: J6.18 (Pin_18), J8.18 (Pin_18)
- new net GPIO3: J5.13 (Pin_13), J7.13 (Pin_13)
- new net GPIO35: J6.13 (Pin_13), J8.13 (Pin_13)
- new net GPIO36: J6.12 (Pin_12), J8.12 (Pin_12)
- new net GPIO37: J6.11 (Pin_11), J8.11 (Pin_11)
- new net GPIO38: J6.10 (Pin_10), J8.10 (Pin_10)
- new net GPIO39: J6.9 (Pin_9), J8.9 (Pin_9)
- new net GPIO40: J6.8 (Pin_8), J8.8 (Pin_8)
- new net GPIO41: J6.7 (Pin_7), J8.7 (Pin_7)
- new net GPIO42: J6.6 (Pin_6), J8.6 (Pin_6)
- new net GPIO45: J6.15 (Pin_15), J8.15 (Pin_15)
- new net GPIO46: J5.14 (Pin_14), J7.14 (Pin_14)
- new net GPIO47: J6.17 (Pin_17), J8.17 (Pin_17)
- new net GPIO48: J6.16 (Pin_16), J8.16 (Pin_16)
- new net GPIO6: J5.6 (Pin_6), J7.6 (Pin_6)
- new net GPIO8: J5.12 (Pin_12), J7.12 (Pin_12)
- new net GPIO9: J5.15 (Pin_15), J7.15 (Pin_15)
- new net LED1: J5.4 (Pin_4), J7.4 (Pin_4), R2.1
- new net LED2: J5.5 (Pin_5), J7.5 (Pin_5), R3.1
- new net REL1: J5.16 (Pin_16), J7.16 (Pin_16), R8.1
- new net REL_COM: J3.1 (Pin_1), K1.1
- new net REL_NA: J3.2 (Pin_2), K1.3
- new net REL_NC: J3.3 (Pin_3), K1.4
- new net RST: J5.3 (Pin_3), J7.3 (Pin_3)
- new net RX0: J6.3 (Pin_3), J8.3 (Pin_3)
- new net SW1: J5.7 (Pin_7), J7.7 (Pin_7), R4.2, SW1.2
- new net SW2: J5.8 (Pin_8), J7.8 (Pin_8), R5.2, SW2.2
- new net TX0: J6.2 (Pin_2), J8.2 (Pin_2)
- new net VIN: C1.1, C6.1, D1.1 (K), U1.3 (VI)
Other:
- note added: "- GPIO0, 3, 45, 46: strapping. GPIO19/20: USB nativo. GPIO43/44: UART0."
- note added: "- GPIO35-37: PSRAM octal en módulos N8R8/N16R8. AN1 en GPIO1 (ADC1)."
- note added: "- LED RGB de la placa: GPIO48 (v1.0) / GPIO38 (v1.1). No usados acá."
- note added: "- Verificar la separación entre tiras con el plano de la DevKit antes del PCB."
- note added: "1: +3V3 2: AN 3: GND"
- note added: "1: CANH 2: CANL 3: GND"
- note added: "1: COM 2: NA 3: NC"
- note added: "3V3"
- note added: "5V"
- note added: "ALIMENTACIÓN (lineal 12 V -> 5 V)"
- note added: "D2: OR con el USB de la DevKit. U1 disipa ~1 W: polígono de cobre +5V en la pestaña (VOUT),"
- note added: "ENTRADA ANALÓGICA 0-10 V (a ADC 0-3,13 V)"
- note added: "ESP32-S3-DevKitC-1 (zócalos hembra 1x22)"
- note added: "EXPANSIÓN (tiras hembra en paralelo con J5 / J6)"
- note added: "GND"
- note added: "GPIO0"
- note added: "GPIO1"
- note added: "GPIO10"
- note added: "GPIO11"
- note added: "GPIO12"
- note added: "GPIO13"
- note added: "GPIO14"
- note added: "GPIO15"
- note added: "GPIO16"
- note added: "GPIO17"
- note added: "GPIO18"
- note added: "GPIO19"
- note added: "GPIO2"
- note added: "GPIO20"
- note added: "GPIO21"
- note added: "GPIO3"
- note added: "GPIO35"
- note added: "GPIO36"
- note added: "GPIO37"
- note added: "GPIO38"
- note added: "GPIO39"
- note added: "GPIO4"
- note added: "GPIO40"
- note added: "GPIO41"
- note added: "GPIO42"
- note added: "GPIO45"
- note added: "GPIO46"
- note added: "GPIO47"
- note added: "GPIO48"
- note added: "GPIO5"
- note added: "GPIO6"
- note added: "GPIO7"
- note added: "GPIO8"
- note added: "GPIO9"
- note added: "Notas DevKit:"
- note added: "PULSADORES"
- note added: "Pin a pin igual que J5/J6 (mismas redes por etiqueta)."
- note added: "RST"
- note added: "RX/44"
- note added: "SALIDA A RELÉ (bobina 5 V)"
- note added: "SALIDAS LED"
- note added: "STBY a GND: modo normal"
- note added: "Si conmuta 220 V: aislar la zona de contactos en el PCB."
- note added: "TRANSCEPTOR CAN"
- note added: "TX/43"
- note added: "U1: 1,25 V x (1 + 390/120) = 5,31 V; después de D2 el riel +5V queda en ~4,9-5,0 V."
- note added: "en ambas caras con vías. C2 tantalio (ESR para estabilidad). R11/R12 dan la carga mínima (~10 mA)."
- title: (none) -> Placa carrier ESP32-S3-DevKitC-1

Commit message: actualiza ruteo con par diferencial
Connections:
- net CANH renamed CAN_P
- net CANL renamed CAN_N
Changed lines of the file:
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@@
 		)
 	)
-	(label "CANH"
+	(label "CAN_P"
 		(at 342.9 181.61 0)
 		(effects
@@
 		)
 	)
-	(label "CANL"
+	(label "CAN_N"
 		(at 340.36 199.39 0)
 		(effects

Commit message: actualiza sch
Connections:
- net GPIO41 is gone; now on net SW2: J6.7 (Pin_7), J8.7 (Pin_7)
- net GPIO42 is gone; now on net SW1: J6.6 (Pin_6), J8.6 (Pin_6)
- net SW1: no longer J5.7 (Pin_7), J7.7 (Pin_7)
- net SW2: no longer J5.8 (Pin_8), J7.8 (Pin_8)
- new net GPIO15: J5.8 (Pin_8), J7.8 (Pin_8)
- new net GPIO7: J5.7 (Pin_7), J7.7 (Pin_7)
Other:
- moved on the sheet: C5, D3, D4, D5, D6, J2, R2, R3, R4, R5, R6, R7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
